Commit message: adding mussel to sim pybullet

File: sim/mussle.urdf (robot description, URDF)
Before this commit: robot urdf_robot, 1 links, 0 joints
Links:
- link base_link: geometry collision sphere radius=0.008; visual mesh filename=pybullet_data/Mussel2.obj

Commit message: easier grab multiple mussels in sim

File: sim/mussle.urdf (robot description, URDF)
Before this commit: robot urdf_robot, 1 links, 0 joints
Links:
- link base_link: geometry collision box size=0.008 0.008 0.048; visual mesh filename=pybullet_data/Mussel2.obj
