Commit message: pybullet bridge start working...

File: sim/brov.urdf (robot description, URDF)
Before this commit: robot myfirst, 4 links, 3 joints
Links:
- removed link left_cm1
- removed link right_cm1
- added link cam1
- added link cam2
- added link left_tube, mass 0.2; visual cylinder length=0.2 radius=0.03
- added link right_tube, mass 0.2; visual cylinder length=0.2 radius=0.03
Joints:
- removed joint base_to_left_cm1
- removed joint base_to_right_cm1
- added joint base_to_cam1: type fixed, parent base_link, child cam1, origin xyz=0.2 0.05 0.0 rpy=0 0 0
- added joint base_to_cam2: type fixed, parent base_link, child cam2, origin xyz=0.2 -0.05 0.0 rpy=0 0 0
- added joint base_to_left_tube: type fixed, parent cm, child left_tube, origin xyz=0.2 -0.05 0.0 rpy=0 0 0
- added joint base_to_right_tube: type fixed, parent cm, child right_tube, origin xyz=0.2 0.05 0.0 rpy=0 0 0
- joint base_to_cm: origin xyz=0 0. 0. rpy=0 1.5707963267948966 0 -> xyz=0 0. 0. rpy=0 0 0

Commit message: pubullet2 based sim is working

File: sim/brov.urdf (robot description, URDF)
Before this commit: robot myfirst, 6 links, 5 joints
Links:
- added link COB, mass 0.0025; visual sphere radius=0.01
- added link COM, mass 0.0025; visual sphere radius=0.01
- link base_link: mass None -> 0.0025
- link cam1: mass None -> 0.0025
- link cam2: mass None -> 0.0025
Joints:
- added joint base_to_cob: type fixed, parent base_link, child COB, origin xyz=0 0. 0.03 rpy=0 0 0
- added joint base_to_com: type fixed, parent base_link, child COM, origin xyz=0 0. -0.03 rpy=0 0 0

Commit message: gripper simulated

File: sim/brov.urdf (robot description, URDF)
Before this commit: robot myfirst, 8 links, 7 joints
Links:
- added link gripper_pole, mass 0.0025; visual cylinder length=0.2 radius=0.01
- added link left_finger, mass 0.0025; visual box size=0.03 .01 0.01
- added link left_finger2, mass 0.0025; visual box size=0.03 0.01 0.01
- added link right_finger, mass 0.0025; visual box size=0.03 0.01 0.01
- added link right_finger2, mass 0.0025; visual box size=0.03 0.01 0.01
Joints:
- added joint gripper_extension: type fixed, parent base_link, child gripper_pole, origin xyz=0.25 0 -0.07 rpy=0 0 0
- added joint gripper_left: type revolute, parent gripper_pole, child left_finger, origin xyz=0.21 0.01 -0.0 rpy=3.1415 0 1, axis 0 0 1, limit lower=0.0 upper=0.548 effort=1000.0 velocity=0.5
- added joint gripper_left2: type fixed, parent left_finger, child left_finger2, origin xyz=0.02 0.01 -0.0 rpy=0 0 1
- added joint gripper_right: type revolute, parent gripper_pole, child right_finger, origin xyz=0.21 -0.01 -0.0 rpy=0 0 -1, axis 0 0 1, limit lower=0.0 upper=0.548 effort=1000.0 velocity=0.5
- added joint gripper_right2: type fixed, parent right_finger, child right_finger2, origin xyz=0.02 0.01 -0.0 rpy=0 0 1

Commit message: update mussle scene

File: sim/brov.urdf (robot description, URDF)
Before this commit: robot myfirst, 13 links, 12 joints
Links:
- link left_finger: geometry collision box size=0.03 0.01 0.01; visual box size=0.03 .01 0.01
- link left_finger2: geometry collision box size=0.03 0.01 0.01; visual box size=0.03 0.01 0.01
- link right_finger: geometry collision box size=0.03 0.01 0.01; visual box size=0.03 0.01 0.01
- link right_finger2: geometry collision box size=0.03 0.01 0.01; visual box size=0.03 0.01 0.01
Joints:
- joint gripper_left: limit lower=0.0 upper=0.548 effort=1000.0 velocity=0.5 -> lower=0.0 upper=0.748 effort=1000.0 velocity=0.5
- joint gripper_right: limit lower=0.0 upper=0.548 effort=1000.0 velocity=0.5 -> lower=0.0 upper=0.748 effort=1000.0 velocity=0.5

Commit message: simulating main camera

File: sim/brov.urdf (robot description, URDF)
Before this commit: robot myfirst, 13 links, 12 joints
Links:
- added link main_cam, mass 0.0025
Joints:
- added joint base_to_main_cam: type fixed, parent base_link, child main_cam, origin xyz=0.2 -0.0 0.3 rpy=0 0 0

Commit message: visable depth image in sim

File: sim/brov.urdf (robot description, URDF)
Before this commit: robot myfirst, 14 links, 13 joints
Links:
- link left_finger: geometry collision box size=0.03 0.01 0.01; visual box size=0.03 0.01 0.01
Joints:
- joint base_to_cam1: origin xyz=0.2 0.05 0.0 rpy=0 0 0 -> xyz=0.2 0.05 -0.15 rpy=0 0 0
- joint base_to_cam2: origin xyz=0.2 -0.05 0.0 rpy=0 0 0 -> xyz=0.2 -0.05 -0.15 rpy=0 0 0
- joint base_to_left_tube: origin xyz=0.2 -0.05 0.0 rpy=0 0 0 -> xyz=0.2 -0.05 -0.15 rpy=0 0 0
- joint base_to_main_cam: origin xyz=0.2 -0.0 0.3 rpy=0 0 0 -> xyz=0.2 -0.0 0.12 rpy=0 0 0
- joint base_to_right_tube: origin xyz=0.2 0.05 0.0 rpy=0 0 0 -> xyz=0.2 0.05 -0.15 rpy=0 0 0
- joint gripper_extension: origin xyz=0.25 0 -0.07 rpy=0 0 0 -> xyz=0.25 0 -0.07 rpy=0 -0.5 0

Commit message: better view of gripper

File: sim/brov.urdf (robot description, URDF)
Before this commit: robot myfirst, 14 links, 13 joints
Joints:
- joint gripper_extension: origin xyz=0.25 0 -0.07 rpy=0 -0.5 0 -> xyz=0.25 0 -0.07 rpy=0 -0.7 0

Commit message: gripper from the side

File: sim/brov.urdf (robot description, URDF)
Before this commit: robot myfirst, 14 links, 13 joints
Joints:
- joint gripper_extension: origin xyz=0.25 0 -0.07 rpy=0 -0.7 0 -> xyz=0.25 0.03 -0.07 rpy=0 -0.7 0

Commit message: tracker track validation

File: sim/brov.urdf (robot description, URDF)
Before this commit: robot myfirst, 14 links, 13 joints
Joints:
- joint gripper_extension: origin xyz=0.25 0.03 -0.07 rpy=0 -0.7 0 -> xyz=0.25 0.03 -0.07 rpy=0 -0.4 0

Commit message: wip

File: sim/brov.urdf (robot description, URDF)
Before this commit: robot myfirst, 14 links, 13 joints
Joints:
- joint base_to_cam1: origin xyz=0.2 0.05 -0.15 rpy=0 0 0 -> xyz=0.2 0.05 0.09 rpy=0 0 0
- joint base_to_cam2: origin xyz=0.2 -0.05 -0.15 rpy=0 0 0 -> xyz=0.2 -0.05 0.09 rpy=0 0 0
- joint base_to_left_tube: origin xyz=0.2 -0.05 -0.15 rpy=0 0 0 -> xyz=0.2 -0.05 0.25 rpy=0 0 0
- joint base_to_right_tube: origin xyz=0.2 0.05 -0.15 rpy=0 0 0 -> xyz=0.2 0.05 0.25 rpy=0 0 0
- joint gripper_extension: origin xyz=0.25 0.03 -0.07 rpy=0 -0.4 0 -> xyz=0.25 0.00 -0.12 rpy=0 -0.4 0

Commit message: update support for rotating gripper

File: sim/brov.urdf (robot description, URDF)
Before this commit: robot myfirst, 14 links, 13 joints
Links:
- added link gripper_pole1, mass 0.0025; visual cylinder length=0.2 radius=0.01
Joints:
- added joint gripper_pole_rotate: type revolute, parent gripper_pole1, child gripper_pole, origin xyz=0.0 0.00 -0.0 rpy=0 0 0, axis 1 0 0, limit lower=-4 upper=4 effort=1000.0 velocity=0.5
- joint gripper_extension: child gripper_pole -> gripper_pole1
